File: MARP_Electrical/SAMD21_TESTING/SAMD21_TESTING.sch (KiCad schematic (older format))
At the start: 3 parts

Commit message: updates_8_15_18
Parts:
- added BT?: 24V Battery, symbol Device:Battery
- added J?: CORTEX_DEBUGGER, symbol Connector_Generic:Conn_02x05_Odd_Even
- added U?: ATSAMD21J18A-AU, QFP50P1200X1200X120_64N, symbol MARP:ATSAMD21J18A-AU
- added U?: LM25017, symbol MARP:LM25017
Connections:
- net labels added: 24V, 3V3, GND, VCC
- wire segments 0 -> 37
- no-connect marks 0 -> 5
