File: MARP_Electrical/MARP/marp_sensory_hub.sch (KiCad schematic (older format))
At the start: 27 parts

Commit message: Added Thermocouple testing project
Parts:
- added J10: PRESS_TRANSD_CH_3, symbol MARP:MOLEX_MINI_FIT_JR_4x4
- added J4: PRESS_TRANSD_CH_0, symbol MARP:MOLEX_MINI_FIT_JR_4x4
- added J6: PRESS_TRANSD_CH_1, symbol MARP:MOLEX_MINI_FIT_JR_4x4
- added J7: PRESS_TRANSD_CH_2, symbol MARP:MOLEX_MINI_FIT_JR_4x4
- added R11, R12, R13, R14, R15, R16, R17, R18: 10k, symbol Device:R
- gave numbers to parts that had none: 27
Connections:
- net GND: now also J10.2 (GND), J10.4 (GND), J4.2 (GND), J4.4 (GND), J6.2 (GND), J6.4 (GND), J7.2 (GND), J7.4 (GND), R12.2, R14.2, R16.2, R18.2
- net at U6.10 (IO4): now also R17.2, R18.1
- net at U6.11 (IO5): now also R15.2, R16.1
- net at U6.12 (IO6): now also R13.2, R14.1
- net at U6.13 (IO7): now also R11.2, R12.1
- new net: J4.1 (DATA), R11.1
- new net: J6.1 (DATA), R13.1
- new net: J7.1 (DATA), R15.1
- new net: J10.1 (DATA), R17.1

Commit message: added a python script for capacitor discharge analysis
Parts:
- renumbered U1 to U4
Changed lines of the file:
@@
 $EndDescr
 $Comp
-L dk_Interface-Sensor-and-Detector-Interfaces:MAX31855KASA_ U1
+L dk_Interface-Sensor-and-Detector-Interfaces:MAX31855KASA_ U4
 U 1 1 5C1953D4
 P 1300 1450
-F 0 "U1" V 1403 709 60  0000 R CNN
+F 0 "U4" V 1403 709 60  0000 R CNN
 F 1 "MAX31855KASA_" V 1297 709 60  0000 R CNN
 F 2 "digikey-footprints:SOIC-8_W3.9mm" H 1500 1650 60  0001 L CNN
@@
 	2000 1250 2300 1250
 $Comp
-L power:GND #PWR017
+L power:GND #PWR023
 U 1 1 5C195745
 P 2300 1250
-F 0 "#PWR017" H 2300 1000 50  0001 C CNN
+F 0 "#PWR023" H 2300 1000 50  0001 C CNN
 F 1 "GND" V 2305 1122 50  0000 R CNN
 F 2 "" H 2300 1250 50  0001 C CNN
@@
 	1200 1350 1000 1350
 $Comp
-L MAX31855:+3V3 #+3V0308
+L MAX31855:+3V3 #+3V08
 U 1 1 5C209C62
 P 900 1350
-F 0 "#+3V0308" H 900 1350 50  0001 C CNN
+F 0 "#+3V08" H 900 1350 50  0001 C CNN
 F 1 "+3V3" V 900 1419 59  0000 L CNN
 F 2 "" H 900 1350 50  0001 C CNN
@@
 	4350 1200 4650 1200
 $Comp
-L power:GND #PWR023
+L power:GND #PWR029
 U 1 1 5C20CFA4
 P 4650 1200
-F 0 "#PWR023" H 4650 950 50  0001 C CNN
+F 0 "#PWR029" H 4650 950 50  0001 C CNN
 F 1 "GND" V 4655 1072 50  0000 R CNN
 F 2 "" H 4650 1200 50  0001 C CNN
@@
 	3550 1300 3350 1300
 $Comp
-L MAX31855:+3V3 #+3V01
+L MAX31855:+3V3 #+3V09
 U 1 1 5C20CFAB
 P 3250 1300
-F 0 "#+3V01" H 3250 1300 50  0001 C CNN
+F 0 "#+3V09" H 3250 1300 50  0001 C CNN
 F 1 "+3V3" V 3250 1369 59  0000 L CNN
 F 2 "" H 3250 1300 50  0001 C CNN
@@
 	6750 1150 7050 1150
 $Comp
-L power:GND #PWR025
+L power:GND #PWR031
 U 1 1 5C20DC3A
 P 7050 1150
-F 0 "#PWR025" H 7050 900 50  0001 C CNN
+F 0 "#PWR031" H 7050 900 50  0001 C CNN
 F 1 "GND" V 7055 1022 50  0000 R CNN
 F 2 "" H 7050 1150 50  0001 C CNN
@@
 	5950 1250 5750 1250
 $Comp
-L MAX31855:+3V3 #+3V02
+L MAX31855:+3V3 #+3V013
 U 1 1 5C20DC41
 P 5650 1250
-F 0 "#+3V02" H 5650 1250 50  0001 C CNN
+F 0 "#+3V013" H 5650 1250 50  0001 C CNN
 F 1 "+3V3" V 5650 1319 59  0000 L CNN
 F 2 "" H 5650 1250 50  0001 C CNN
@@
 	9200 1150 9500 1150
 $Comp
-L power:GND #PWR026
+L power:GND #PWR032
 U 1 1 5C20E7D1
 P 9500 1150
-F 0 "#PWR026" H 9500 900 50  0001 C CNN
+F 0 "#PWR032" H 9500 900 50  0001 C CNN
 F 1 "GND" V 9505 1022 50  0000 R CNN
 F 2 "" H 9500 1150 50  0001 C CNN
@@
 	8400 1250 8200 1250
 $Comp
-L MAX31855:+3V3 #+3V03
+L MAX31855:+3V3 #+3V014
 U 1 1 5C20E7D8
 P 8100 1250
-F 0 "#+3V03" H 8100 1250 50  0001 C CNN
+F 0 "#+3V014" H 8100 1250 50  0001 C CNN
 F 1 "+3V3" V 8100 1319 59  0000 L CNN
 F 2 "" H 8100 1250 50  0001 C CNN
@@
 	4200 5200 4200 5250
 $Comp
-L power:GND #PWR021
+L power:GND #PWR027
 U 1 1 5C2169AA
 P 4200 5250
-F 0 "#PWR021" H 4200 5000 50  0001 C CNN
+F 0 "#PWR027" H 4200 5000 50  0001 C CNN
 F 1 "GND" H 4205 5077 50  0000 C CNN
 F 2 "" H 4200 5250 50  0001 C CNN
@@
 Connection ~ 4200 4900
 $Comp
-L MAX31855:+3V3 #+3V03011
+L MAX31855:+3V3 #+3V012
 U 1 1 5C218CC1
 P 4750 4900
-F 0 "#+3V03011" H 4750 4900 50  0001 C CNN
+F 0 "#+3V012" H 4750 4900 50  0001 C CNN
 F 1 "+3V3" V 4750 4969 59  0000 L CNN
 F 2 "" H 4750 4900 50  0001 C CNN
@@
 	4300 4300 4750 4300
 $Comp
-L power:GND #PWR024
+L power:GND #PWR030
 U 1 1 5C221E10
 P 5200 4200
-F 0 "#PWR024" H 5200 3950 50  0001 C CNN
+F 0 "#PWR030" H 5200 3950 50  0001 C CNN
 F 1 "GND" H 5205 4027 50  0000 C CNN
 F 2 "" H 5200 4200 50  0001 C CNN
@@
 	4600 4100 4600 3900
 $Comp
-L MAX31855:+3V3 #+3V03010
+L MAX31855:+3V3 #+3V011
 U 1 1 5C2D8E3F
 P 4600 3800
-F 0 "#+3V03010" H 4600 3800 50  0001 C CNN
+F 0 "#+3V011" H 4600 3800 50  0001 C CNN
 F 1 "+3V3" H 4600 3921 59  0000 C CNN
 F 2 "" H 4600 3800 50  0001 C CNN
@@
 $EndComp
 $Comp
-L MAX31855:+3V3 #+3V0309
+L MAX31855:+3V3 #+3V010
 U 1 1 5C2D8EB2
 P 3500 5000
-F 0 "#+3V0309" H 3500 5000 50  0001 C CNN
+F 0 "#+3V010" H 3500 5000 50  0001 C CNN
 F 1 "+3V3" V 3500 5069 59  0000 L CNN
 F 2 "" H 3500 5000 50  0001 C CNN
@@
 $EndComp
 $Comp
-L power:GND #PWR010
+L power:GND #PWR021
 U 1 1 5C35D652
 P 1800 3450
-F 0 "#PWR010" H 1800 3200 50  0001 C CNN
+F 0 "#PWR021" H 1800 3200 50  0001 C CNN
 F 1 "GND" V 1805 3322 50  0000 R CNN
 F 2 "" H 1800 3450 50  0001 C CNN
@@
 	800  4650 800  4750
 $Comp
-L power:GND #PWR06
+L power:GND #PWR019
 U 1 1 5C372925
 P 800 4750
-F 0 "#PWR06" H 800 4500 50  0001 C CNN
+F 0 "#PWR019" H 800 4500 50  0001 C CNN
 F 1 "GND" H 805 4577 50  0000 C CNN
 F 2 "" H 800 4750 50  0001 C CNN
@@
 $EndComp
 $Comp
-L power:GND #PWR018
+L power:GND #PWR024
 U 1 1 5C375389
 P 2350 4400
-F 0 "#PWR018" H 2350 4150 50  0001 C CNN
+F 0 "#PWR024" H 2350 4150 50  0001 C CNN
 F 1 "GND" V 2355 4272 50  0000 R CNN
 F 2 "" H 2350 4400 50  0001 C CNN
@@
 	1350 5600 1350 5700
 $Comp
-L power:GND #PWR08
+L power:GND #PWR020
 U 1 1 5C3753A8
 P 1350 5700
-F 0 "#PWR08" H 1350 5450 50  0001 C CNN
+F 0 "#PWR020" H 1350 5450 50  0001 C CNN
 F 1 "GND" H 1355 5527 50  0000 C CNN
 F 2 "" H 1350 5700 50  0001 C CNN
@@
 $EndComp
 $Comp
-L power:GND #PWR019
+L power:GND #PWR025
 U 1 1 5C3807BB
 P 2800 5600
-F 0 "#PWR019" H 2800 5350 50  0001 C CNN
+F 0 "#PWR025" H 2800 5350 50  0001 C CNN
 F 1 "GND" V 2805 5472 50  0000 R CNN
 F 2 "" H 2800 5600 50  0001 C CNN
@@
 	1800 6800 1800 6900
 $Comp
-L power:GND #PWR016
+L power:GND #PWR022
 U 1 1 5C3807D9
 P 1800 6900
-F 0 "#PWR016" H 1800 6650 50  0001 C CNN
+F 0 "#PWR022" H 1800 6650 50  0001 C CNN
 F 1 "GND" H 1805 6727 50  0000 C CNN
 F 2 "" H 1800 6900 50  0001 C CNN
@@
 $EndComp
 $Comp
-L power:GND #PWR022
+L power:GND #PWR028
 U 1 1 5C389125
 P 4350 6200
-F 0 "#PWR022" H 4350 5950 50  0001 C CNN
+F 0 "#PWR028" H 4350 5950 50  0001 C CNN
 F 1 "GND" V 4355 6072 50  0000 R CNN
 F 2 "" H 4350 6200 50  0001 C CNN
@@
 	3350 7400 3350 7500
 $Comp
-L power:GND #PWR020
+L power:GND #PWR026
 U 1 1 5C389143
 P 3350 7500
-F 0 "#PWR020" H 3350 7250 50  0001 C CNN
+F 0 "#PWR026" H 3350 7250 50  0001 C CNN
 F 1 "GND" H 3355 7327 50  0000 C CNN
 F 2 "" H 3350 7500 50  0001 C CNN
