File: MARP_Electrical/MARP/MARP.sch (KiCad schematic (older format))
At the start: 35 parts, among them J1 MOLEX_47219-2001, J2 CORTEX_DEBUGGER, P1 292304-1, Q1 FQP27P06, Q2 FQP27P06, U1 FT232RL, U2 ATSAMD21J18A-AU, U3 XBP9B-XCWT-002

Commit message: Removed a lot. Starting over on some things
Parts:
- removed C1: 10nF, symbol Device:CP1_Small
- removed C2, C3, C4, C5, C7: 100nF, symbol Device:C_Small
- removed C6: 1uF, symbol Device:C_Small
- removed C8: 10uF, symbol Device:C_Small
- removed D1, D6: LED, symbol Device:LED
- removed D2: USB_RX_LED, symbol Device:LED
- removed D3: USB_TX_LED, symbol Device:LED
- removed D4: XBEE TX LED, symbol Device:LED
- removed D5: XBEE RX LED, symbol Device:LED
- removed J2: CORTEX_DEBUGGER, symbol Connector_Generic:Conn_02x05_Odd_Even
- removed L1: Ferrite_Bead_Small, symbol Device:Ferrite_Bead_Small
- removed L2: 220OHM, symbol Device:Ferrite_Bead_Small
- removed P1: 292304-1, symbol MARP-rescue:292304-1-Connector
- removed Q1, Q2: FQP27P06, digikey-footprints:TO-92-3, symbol dk_Transistors-FETs-MOSFETs-Single:FQP27P06
- removed R1: 4700, symbol Device:R_Small
- removed R10, R7: 10k, symbol Device:R_Small
- removed R2: 2200, symbol Device:R_Small
- removed R3, R4, R5, R6, R8: 330, symbol Device:R_Small
- removed R9: R_Small, symbol Device:R_Small
- removed S1: GPTS203211B, digikey-footprints:PushButton_12x12mm_THT_GPTS203211B, symbol dk_Pushbutton-Switches:GPTS203211B
- removed U1: FT232RL, Package_SO:SSOP-28_5.3x10.2mm_P0.65mm, symbol Interface_USB:FT232RL
- removed U2: ATSAMD21J18A-AU, symbol MARP:ATSAMD21J18A-AU
- removed U3: XBP9B-XCWT-002, symbol XBEE_900HP:XBP9B-XCWT-002
- added C? (x6): 10nF, symbol Device:C
- added C?: 1uF, symbol Device:C_Small
- added C? (x3): 100nF, symbol Device:C_Small
- added C?: 10uF, symbol Device:C_Small
- added D? (x6): DIODE, symbol pspice:DIODE
- added FB? (x12): 470OHM, symbol Device:Ferrite_Bead_Small
- added J?: TP0_1_P, symbol Connector:Conn_01x01_Male
- added J?: TP0_1_N, symbol Connector:Conn_01x01_Male
- added J?: TP1_1_P, symbol Connector:Conn_01x01_Male
- added J?: TP1_1_N, symbol Connector:Conn_01x01_Male
- added J?: TP2_1_P, symbol Connector:Conn_01x01_Male
- added J?: TP2_1_N, symbol Connector:Conn_01x01_Male
- added J? (x3): TP3_1_P, symbol Connector:Conn_01x01_Male
- added J? (x3): TP3_1_N, symbol Connector:Conn_01x01_Male
- added J?: PT_0, symbol MARP:Press_Transducer_Header
- added J?: PT_1, symbol MARP:Press_Transducer_Header
- added J?: PT_2, symbol MARP:Press_Transducer_Header
- added J?: PT_3, symbol MARP:Press_Transducer_Header
- added J? (x4): Press_Transducer_Header, symbol MARP:Press_Transducer_Header
- added K?: 24V_GP_RELAY_1, Relay_THT:Relay_SPDT_SANYOU_SRD_Series_Form_C, symbol Relay:SANYOU_SRD_Form_C
- added K?: 24V_GP_RELAY_0, Relay_THT:Relay_SPDT_SANYOU_SRD_Series_Form_C, symbol Relay:SANYOU_SRD_Form_C
- added K? (x3): 12V_GP_RELAY_0, Relay_THT:Relay_SPDT_SANYOU_SRD_Series_Form_C, symbol Relay:SANYOU_SRD_Form_C
- added K?: 24V_GP_RELAY_2, Relay_THT:Relay_SPDT_SANYOU_SRD_Series_Form_C, symbol Relay:SANYOU_SRD_Form_C
- added L?: 220OHM, symbol Device:Ferrite_Bead_Small
- added Q? (x6): GP_RELAY_NFET, digikey-footprints:TO-92-3, symbol MARP-rescue:FQP27P06-dk_Transistors-FETs-MOSFETs-Single
- added R? (x6): 10k, symbol Device:R
- added TH? (x6): Thermistor, symbol Device:Thermistor
- added U? (x6): MAX31855KASA_, digikey-footprints:SOIC-8_W3.9mm, symbol MARP-rescue:MAX31855KASA_-dk_Interface-Sensor-and-Detector-Interfaces
- added U?: AD5593R, Package_SO:TSSOP-16_4.4x5mm_P0.65mm, symbol Analog:AD5593R
- added U?: D21_DAQ_AND_HEALTH_MONITORING, symbol MARP:ATSAMD21J18A-AU
- J1: symbol MOLEX_47219-2001:MOLEX_47219-2001 -> MARP-rescue:MOLEX_47219-2001-MOLEX_47219-2001
Connections:
- net GND: now also C?.1, C?.1, C?.1, C?.2, C?.2, Q?.3 (S), Q?.3 (S), Q?.3 (S), Q?.3 (S), Q?.3 (S), Q?.3 (S), R?.2, R?.2, R?.2, R?.2, R?.2, R?.2, U?.1 (GND), U?.1 (GND), U?.1 (GND), U?.1 (GND), U?.1 (GND), U?.1 (GND), U?.22 (GND), U?.33 (GND), U?.47 (GND), U?.54 (GND), U?.7 (GNDANA); no longer J1.6 (GND), J1.G1 (1_GND), J1.G2 (2_GND), J1.G3 (3_GND), J1.G4 (4_GND)
- net SPI0_SCK: now also U?.5 (SCK), U?.5 (SCK), U?.5 (SCK), U?.5 (SCK), U?.5 (SCK), U?.5 (SCK); no longer J1.5 (SCLK)
- net ~SPI0_THERMO0_SS: now also U?.6 (~CS)
- net ~SPI0_THERMO1_SS: now also U?.6 (~CS)
- net ~SPI0_THERMO2_SS: now also U?.6 (~CS)
- net ~SPI0_THERMO3_SS: now also U?.6 (~CS)
- net SPI0_MISO: no longer names the net of J1.7 (DO)
- net SPI0_MOSI: no longer names the net of J1.3 (DI)
- net ~SPI0_SDCARD_SS: no longer names the net of J1.2 (CS)
- new net: C?.2, FB?.1, U?.2 (T-) (x6)
- new net: C?.1, FB?.1, U?.3 (T+) (x6)
- new net: FB?.2, J?.1 (Pin_1) (x12)
- new net: D?.1 (K), K?.2, Q?.2 (D) (x6)
- new net: C?.2, U?.55 (VDDCORE)
- new net: C?.1, C?.1, C?.2, C?.2, L?.1, U?.21 (VDDIO), U?.34 (VDDIO), U?.48 (VDDIO), U?.56 (VDDIN)
- new net: L?.2, U?.8 (VDDANA)
- new net +5V: D?.2 (A), D?.2 (A), D?.2 (A), D?.2 (A), D?.2 (A), D?.2 (A), K?.5, K?.5, K?.5, K?.5, K?.5, K?.5
- new net SIG_12V_RELAY_0: Q?.1 (G), Q?.1 (G), R?.1, R?.1
- new net SIG_12V_RELAY_1: Q?.1 (G), R?.1
- new net SIG_24V_RELAY_0: Q?.1 (G), R?.1
- new net SIG_24V_RELAY_1: Q?.1 (G), R?.1
- new net SIG_24V_RELAY_2: Q?.1 (G), R?.1
- new net SPI0_SO: U?.7 (SO), U?.7 (SO), U?.7 (SO), U?.7 (SO), U?.7 (SO), U?.7 (SO)
- new net ~SPI0_THERMO4_SS: U?.6 (~CS)
- new net ~SPI0_THERMO5_SS: U?.6 (~CS)
- no-connect marks 6 -> 2
Other:
- note added: "BRAIN"
- note added: "DAQ HUB"
- note added: "GEN PURPOSE HUB"
- note added: "PRESSURE TRANSDUCER HUB"
- note added: "THERMOCOUPLE HUB"

Commit message: excel sheet + some rpicm3 modules
Parts:
- removed J1: MOLEX_47219-2001, symbol MARP-rescue:MOLEX_47219-2001-MOLEX_47219-2001
- removed J? (x4): Press_Transducer_Header, symbol MARP:Press_Transducer_Header
- removed TH? (x5): Thermistor, symbol Device:Thermistor
- added C? (x2): 220nF, symbol Device:C_Small
- added D? (x2): DIODE, symbol pspice:DIODE
- added J?: PT_7, symbol MARP:Press_Transducer_Header
- added J?: PT_6, symbol MARP:Press_Transducer_Header
- added J?: PT_5, symbol MARP:Press_Transducer_Header
- added J?: PT_4, symbol MARP:Press_Transducer_Header
- added J?: Conn_ARM_JTAG_SWD_10, Connector_PinHeader_1.27mm:PinHeader_2x05_P1.27mm_Vertical_SMD, symbol Connector:Conn_ARM_JTAG_SWD_10
- added J? (x2): USB_A, symbol Connector:USB_A
- added J?: Wuerth_7499010121A, Connector_RJ:RJ45_Wuerth_7499010121A_Horizontal, symbol Connector:Wuerth_7499010121A
- added K?: 5V_GP_RELAY_0, Relay_THT:Relay_SPDT_SANYOU_SRD_Series_Form_C, symbol Relay:SANYOU_SRD_Form_C
- added K?: 5V_GP_RELAY_1, Relay_THT:Relay_SPDT_SANYOU_SRD_Series_Form_C, symbol Relay:SANYOU_SRD_Form_C
- added Q? (x2): GP_RELAY_NFET, digikey-footprints:TO-92-3, symbol MARP-rescue:FQP27P06-dk_Transistors-FETs-MOSFETs-Single
- added R? (x8): R_Small, symbol Device:R_Small
- added R? (x16): 10k, symbol Device:R_Small
- added R? (x2): 10k, symbol Device:R
- added TH?: SYS_MON_THERM_1, symbol Device:Thermistor
- added TH?: SYS_MON_THERM_2, symbol Device:Thermistor
- added TH?: SYS_MON_THERM_3, symbol Device:Thermistor
- added TH?: SYS_MON_THERM_4, symbol Device:Thermistor
- added TH?: SYS_MON_THERM_5, symbol Device:Thermistor
- added U? (x2): LAN9512, Package_DFN_QFN:QFN-64-1EP_9x9mm_P0.5mm_EP7.3x7.3mm, symbol Interface_Ethernet:LAN9512
- added U? (x2): HUMIDITY_SENS_0, symbol MARP:MS8607
- added U?: XBP9B-XCWT-002-XBEE_900HP, DIP2200W51P200L3294H279Q20P, symbol MARP:XBP9B-XCWT-002-XBEE_900HP
- added U?: ENC28J60x-ML, Package_DFN_QFN:QFN-28-1EP_6x6mm_P0.65mm_EP4.25x4.25mm, symbol Interface_Ethernet:ENC28J60x-ML
- K?: value 12V_GP_RELAY_0 -> 12V_GP_RELAY_1
- K?: value 12V_GP_RELAY_0 -> 12V_GP_RELAY_2
- TH?: value Thermistor -> SYS_MON_THERM_0
Connections:
- net +5V: now also J?.1 (5V+), J?.1 (5V+), J?.1 (5V+), J?.1 (5V+), D?.2 (A), D?.2 (A), J?.1 (5V+), J?.1 (5V+), J?.1 (5V+), J?.1 (5V+), K?.5, K?.5
- net GND: now also J?.2 (GND), J?.2 (GND), J?.2 (GND), J?.2 (GND), J?.3 (GND), J?.3 (GND), J?.3 (GND), J?.3 (GND), TH?.1, U?.14 (GND), U?.2 (A0), J?.2 (GND), J?.2 (GND), J?.2 (GND), J?.2 (GND), J?.3 (GND), J?.3 (GND), J?.3 (GND), J?.3 (GND), Q?.3 (S), Q?.3 (S), R?.2, R?.2, R?.2, R?.2, R?.2, R?.2, R?.2, R?.2, R?.2, R?.2, TH?.1, TH?.1, TH?.1, TH?.1, TH?.1
- net SIG_12V_RELAY_0: no longer Q?.1 (G), R?.1
- net SPI0_SCK: now also U?.50 (PB23)
- net SPI0_SO: now also U?.49 (PB22)
- net SYS_MON_ADC_0: now reaches TH?.2
- net SYS_MON_ADC_0: now also U?.3 (PA02), R?.2
- net at J?.4 (SIG): now also R?.2 (x4)
- net at U?.10 (IO4): now also R?.1, R?.2
- net at U?.11 (IO5): now also R?.1, R?.2
- net at U?.12 (IO6): now also R?.1, R?.2
- net at U?.13 (IO7): now also R?.1, R?.2
- net at U?.4 (IO0): now also R?.1, R?.1
- net at U?.5 (IO1): now also R?.1, R?.1
- net at U?.6 (IO2): now also R?.1, R?.1
- net at U?.7 (IO3): now also R?.1, R?.1
- net SYS_MON_ADC_2: now reaches U?.11 (PB08)
- net SYS_MON_ADC_2: now also R?.2, TH?.2
- net SYS_MON_ADC_3: now reaches U?.12 (PB09)
- net SYS_MON_ADC_3: now also R?.2, TH?.2
- net SYS_MON_ADC_4: now reaches U?.13 (PA04)
- net SYS_MON_ADC_4: now also R?.2, TH?.2
- net SYS_MON_ADC_5: now reaches U?.14 (PA05)
- net SYS_MON_ADC_5: now also R?.2, TH?.2
- net BRAIN_SDA: now reaches U?.17 (PA08)
- net BRAIN_SDA: now also U?.7 (SDA)
- net BRAIN_SCL: now reaches U?.18 (PA09)
- net BRAIN_SCL: now also U?.8 (SCL)
- net SYS_MON_ADC_1: now reaches U?.4 (PA03)
- net SYS_MON_ADC_1: now also R?.2, TH?.2
- net DAQ_I2C_SDA: now reaches U?.43 (PA22)
- net DAQ_I2C_SDA: now also R?.2, U?.7 (SDA)
- net DAQ_I2C_SCL: now reaches U?.44 (PA23)
- net DAQ_I2C_SCL: now also R?.2, U?.8 (SCL)
- new net: U?.10 (VDD33A), U?.49 (VDD33A), U?.5 (VDD33A), U?.51 (VDD33A), U?.54 (VDD33A), U?.57 (VDD33A), U?.64 (VDD33A)
- new net: U?.15 (VDD18CORE), U?.38 (VDD18CORE)
- new net: U?.19 (VDD33IO), U?.27 (VDD33IO), U?.33 (VDD33IO), U?.39 (VDD33IO), U?.46 (VDD33IO)
- new net: J?.4 (SIG), R?.1 (x4)
- new net: D?.1 (K), K?.2, Q?.2 (D) (x2)
- new net: C?.2, U?.3 (GND) (x2)
- new net: J?.3 (GND), J?.5 (GND)
- new net +3V3: C?.1, C?.1, R?.1, R?.1, R?.1, R?.1, R?.1, R?.1, R?.1, R?.1, U?.1 (VDD), U?.1 (VDD)
- new net SIG_12V_RELAY_2: Q?.1 (G), R?.1
- new net SIG_5V_RELAY_0: Q?.1 (G), R?.1
- new net SIG_5V_RELAY_1: Q?.1 (G), R?.1
- no-connect marks 2 -> 4
Other:
- note added: "900MHz XBEE"
- note added: "COMMUNICATIONS HUB"
- note added: "DAQ BRAIN"
- note added: "ETHERNET"
- note added: "SYSTEM MONITORING"
- note added: "USB"
- note removed: "BRAIN"
- note removed: "DAQ HUB"
- moved on the sheet: C?, D?, FB?, J?, K?, L?, Q?, R?, TH?, U?

Commit message: Updated schematic
Connections:
- net BRAIN_SCL: no longer U?.8 (SCL)
- net BRAIN_SDA: no longer U?.7 (SDA)
- net DAQ_I2C_SCL: now also U?.8 (SCL)
- net DAQ_I2C_SDA: now also U?.7 (SDA)
Other:
- note added: "DAQ HEALTH MON BRAIN"
- note removed: "DAQ BRAIN"
Changed lines of the file:
@@
 $EndComp
 Text Notes 19650 20300 0    394  ~ 0
-DAQ BRAIN
+DAQ HEALTH MON BRAIN
 $Comp
 L MARP-rescue:MAX31855KASA_-dk_Interface-Sensor-and-Detector-Interfaces U?
@@
 Wire Wire Line
 	29350 21850 29200 21850
-Text GLabel 29200 21750 0    50   Input ~ 0
-BRAIN_SDA
-Text GLabel 29200 21850 0    50   Input ~ 0
-BRAIN_SCL
 $Comp
 L Connector:Conn_ARM_JTAG_SWD_10 J?
@@
 Text Notes 12250 2650 0    236  ~ 0
 900MHz XBEE
+Text GLabel 29200 21750 0    50   Input ~ 0
+DAQ_I2C_SDA
+Text GLabel 29200 21850 0    50   Input ~ 0
+DAQ_I2C_SCL
 $EndSCHEMATC
