File: MARP_Electrical/MARP/MARP.sch (KiCad schematic (older format))
At the start: 126 parts

Commit message: Updated schematic
Parts:
- U?: value HUMIDITY_SENS_0 -> HUMIDITY_SENS_1
Other:
- note added: "DAQ SYS MON BRAIN"
- note removed: "DAQ HEALTH MON BRAIN"
Changed lines of the file:
@@
 	1    0    0    -1
 $EndComp
-Text Notes 19650 20300 0    394  ~ 0
-DAQ HEALTH MON BRAIN
+Text Notes 17650 20050 0    394  ~ 0
+DAQ SYS MON BRAIN
 $Comp
 L MARP-rescue:MAX31855KASA_-dk_Interface-Sensor-and-Detector-Interfaces U?
@@
 P 29550 21700
 F 0 "U?" H 29728 21746 50  0000 L CNN
-F 1 "HUMIDITY_SENS_0" H 29728 21655 50  0000 L CNN
+F 1 "HUMIDITY_SENS_1" H 29728 21655 50  0000 L CNN
 F 2 "" H 29150 21650 50  0001 C CNN
 F 3 "" H 29150 21650 50  0001 C CNN

Commit message: Updated schematic
Parts:
- added U?: AS8506C, Package_DFN_QFN:QFN-40-1EP_6x6mm_P0.5mm_EP4.6x4.6mm, symbol Battery_Management:AS8506C
Changed lines of the file:
@@
 Text GLabel 29200 21850 0    50   Input ~ 0
 DAQ_I2C_SCL
+$Comp
+L Battery_Management:AS8506C U?
+U 1 1 5C9B506A
+P 14050 14800
+F 0 "U?" H 14050 13914 50  0000 C CNN
+F 1 "AS8506C" H 14050 13823 50  0000 C CNN
+F 2 "Package_DFN_QFN:QFN-40-1EP_6x6mm_P0.5mm_EP4.6x4.6mm" H 14050 14800 50  0001 C CNN
+F 3 "http://ams.com/eng/content/download/476603/1402377/252935" H 13100 15000 50  0001 C CNN
+	1    14050 14800
+	1    0    0    -1
+$EndComp
 $EndSCHEMATC

Commit message: deleted random part
Parts:
- removed U?: AS8506C, Package_DFN_QFN:QFN-40-1EP_6x6mm_P0.5mm_EP4.6x4.6mm, symbol Battery_Management:AS8506C
Changed lines of the file:
@@
 Text GLabel 29200 21850 0    50   Input ~ 0
 DAQ_I2C_SCL
-$Comp
-L Battery_Management:AS8506C U?
-U 1 1 5C9B506A
-P 14050 14800
-F 0 "U?" H 14050 13914 50  0000 C CNN
-F 1 "AS8506C" H 14050 13823 50  0000 C CNN
-F 2 "Package_DFN_QFN:QFN-40-1EP_6x6mm_P0.5mm_EP4.6x4.6mm" H 14050 14800 50  0001 C CNN
-F 3 "http://ams.com/eng/content/download/476603/1402377/252935" H 13100 15000 50  0001 C CNN
-	1    14050 14800
-	1    0    0    -1
-$EndComp
 $EndSCHEMATC

Commit message: Associated thing
Parts:
- U10: renamed from U?; footprint (none) -> Package_QFP:LQFP-64_10x10mm_P0.5mm
- gave numbers to parts that had none: 124

Commit message: .
Parts:
- U3, U4, U5, U6, U8, U9: footprint digikey-footprints:SOIC-8_W3.9mm -> marp:Thermocouple_Connector_PCC-SMP-K
- U7: footprint DIP2200W51P200L3294H279Q20P -> (none)
Changed lines of the file:
@@
 F 0 "U3" V 5103 30309 60  0000 R CNN
 F 1 "MAX31855KASA_" V 4997 30309 60  0000 R CNN
-F 2 "digikey-footprints:SOIC-8_W3.9mm" H 5200 31250 60  0001 L CNN
+F 2 "marp:Thermocouple_Connector_PCC-SMP-K" H 5200 31250 60  0001 L CNN
 F 3 "https://datasheets.maximintegrated.com/en/ds/MAX31855.pdf" H 5200 31350 60  0001 L CNN
 F 4 "MAX31855KASA+-ND" H 5200 31450 60  0001 L CNN "Digi-Key_PN"
@@
 F 0 "U4" V 7453 30259 60  0000 R CNN
 F 1 "MAX31855KASA_" V 7347 30259 60  0000 R CNN
-F 2 "digikey-footprints:SOIC-8_W3.9mm" H 7550 31200 60  0001 L CNN
+F 2 "marp:Thermocouple_Connector_PCC-SMP-K" H 7550 31200 60  0001 L CNN
 F 3 "https://datasheets.maximintegrated.com/en/ds/MAX31855.pdf" H 7550 31300 60  0001 L CNN
 F 4 "MAX31855KASA+-ND" H 7550 31400 60  0001 L CNN "Digi-Key_PN"
@@
 F 0 "U5" V 9853 30209 60  0000 R CNN
 F 1 "MAX31855KASA_" V 9747 30209 60  0000 R CNN
-F 2 "digikey-footprints:SOIC-8_W3.9mm" H 9950 31150 60  0001 L CNN
+F 2 "marp:Thermocouple_Connector_PCC-SMP-K" H 9950 31150 60  0001 L CNN
 F 3 "https://datasheets.maximintegrated.com/en/ds/MAX31855.pdf" H 9950 31250 60  0001 L CNN
 F 4 "MAX31855KASA+-ND" H 9950 31350 60  0001 L CNN "Digi-Key_PN"
@@
 F 0 "U6" V 12303 30209 60  0000 R CNN
 F 1 "MAX31855KASA_" V 12197 30209 60  0000 R CNN
-F 2 "digikey-footprints:SOIC-8_W3.9mm" H 12400 31150 60  0001 L CNN
+F 2 "marp:Thermocouple_Connector_PCC-SMP-K" H 12400 31150 60  0001 L CNN
 F 3 "https://datasheets.maximintegrated.com/en/ds/MAX31855.pdf" H 12400 31250 60  0001 L CNN
 F 4 "MAX31855KASA+-ND" H 12400 31350 60  0001 L CNN "Digi-Key_PN"
@@
 F 0 "U8" V 14653 30159 60  0000 R CNN
 F 1 "MAX31855KASA_" V 14547 30159 60  0000 R CNN
-F 2 "digikey-footprints:SOIC-8_W3.9mm" H 14750 31100 60  0001 L CNN
+F 2 "marp:Thermocouple_Connector_PCC-SMP-K" H 14750 31100 60  0001 L CNN
 F 3 "https://datasheets.maximintegrated.com/en/ds/MAX31855.pdf" H 14750 31200 60  0001 L CNN
 F 4 "MAX31855KASA+-ND" H 14750 31300 60  0001 L CNN "Digi-Key_PN"
@@
 F 0 "U9" V 16953 30059 60  0000 R CNN
 F 1 "MAX31855KASA_" V 16847 30059 60  0000 R CNN
-F 2 "digikey-footprints:SOIC-8_W3.9mm" H 17050 31000 60  0001 L CNN
+F 2 "marp:Thermocouple_Connector_PCC-SMP-K" H 17050 31000 60  0001 L CNN
 F 3 "https://datasheets.maximintegrated.com/en/ds/MAX31855.pdf" H 17050 31100 60  0001 L CNN
 F 4 "MAX31855KASA+-ND" H 17050 31200 60  0001 L CNN "Digi-Key_PN"
@@
 F 0 "U7" H 13450 5067 50  0000 C CNN
 F 1 "XBP9B-XCWT-002-XBEE_900HP" H 13450 4976 50  0000 C CNN
-F 2 "DIP2200W51P200L3294H279Q20P" H 13450 4000 50  0001 L BNN
+F 2 "" H 13450 4000 50  0001 L BNN
 F 3 "Xbee-Pro Xsc S3b, 900 Mhz, 250mw, Wire Antenna, 19.2 Kbps" H 13450 4000 50  0001 L BNN
 F 4 "Digi International" H 13450 4000 50  0001 L BNN "Field4"
